File: PCB/linkytic/_autosave-linkytic.kicad_sch (KiCad schematic)
At the start: 34 parts, among them J1 L2, J2 L1, J3 A, SW1 benoit, U1 M5333B, U2 E18-MS1-PCB, U3 CC_debugger

Commit message: save before usb adding, last modif
Parts:
- U4: renamed from U?; footprint (none) -> Package_SO:SOP-8_5.28x5.23mm_P1.27mm
- gave numbers to parts that had none: 19
