File: PCB/linkytic/linkytic.kicad_sch (KiCad schematic)
At the start: 34 parts, among them J1 L2, J2 L1, J3 A, SW1 benoit, U1 M5333B, U2 E18-MS1-PCB, U3 CC_debugger

Commit message: Update final version V0
Parts:
- removed C?: CP_Radial_D8.0mm_P2.50mm, Capacitor_THT_AKL:CP_Radial_D8.0mm_P2.50mm, symbol Capacitor_AKL:CP_Radial_D8.0mm_P2.50mm
- added C3: 1u, Capacitor_SMD:C_0603_1608Metric, symbol Device:C
- added J6: USB_B_Micro, usb:USB_aliexpress, symbol Connector:USB_B_Micro
- C4: renamed from C?; value 4.7uF -> 10uF
- J4, J5: renamed from J?; footprint (none) -> Connector_PinHeader_1.27mm:PinHeader_1x01_P1.27mm_Vertical
- U4: renamed from U?; footprint (none) -> Package_SO:SOP-8_3.76x4.96mm_P1.27mm
- gave numbers to parts that had none: 15
Connections:
- net GND_2: now also U4.1 (TEMP), C3.2, J6.5 (GND), J6.6 (Shield)
- net USB_IN: now also J6.1 (VBUS)
- net at D4.1 (K), Q1.2 (S), U5.2 (VIN): now also C3.1
